Commit message: zed urdf

File: zed_ws/src/zed-ros-wrapper/urdf/zed.urdf (robot description, URDF)
Before this commit: robot zed_camera, 4 links, 3 joints
Links:
- added link zed_hinge
Joints:
- added joint zed_hinge_joint: type fixed, parent zed_hinge, child zed_center, origin xyz=0 0 0 rpy=0 -0.52 0
